Commit message: Modify STL name

File: rosbook_ws/src/ch18_22_robot_arm/urdf/robot_arm.urdf (robot description, URDF)
Before this commit: robot jdcobot_100_description, 7 links, 6 joints
Links:
- link base_link: geometry collision mesh filename=package://ch18_22_robot_arm/meshes/base.stl; visual mesh filename=package://ch18_22_robot_arm/meshes/base.stl
- link link_1: geometry collision mesh filename=package://ch18_22_robot_arm/meshes/shoulder_big_part_1.stl; visual mesh filename=package://ch18_22_robot_arm/meshes/shoulder_big_part_1.stl
- link link_2: geometry collision mesh filename=package://ch18_22_robot_arm/meshes/shoulder_elbow.stl; visual mesh filename=package://ch18_22_robot_arm/meshes/shoulder_elbow.stl
- link link_3: geometry collision mesh filename=package://ch18_22_robot_arm/meshes/elbow_wrist.stl; visual mesh filename=package://ch18_22_robot_arm/meshes/elbow_wrist.stl
- link link_4: geometry collision mesh filename=package://ch18_22_robot_arm/meshes/wrist_assembly.stl; visual mesh filename=package://ch18_22_robot_arm/meshes/wrist_assembly.stl
- link link_5: geometry collision mesh filename=package://ch18_22_robot_arm/meshes/Round_gear.stl; visual mesh filename=package://ch18_22_robot_arm/meshes/Round_gear.stl
- link link_6: geometry collision mesh filename=package://ch18_22_robot_arm/meshes/gripper_finger.stl; visual mesh filename=package://ch18_22_robot_arm/meshes/gripper_finger.stl
Joints:
- removed joint joint_1
- removed joint joint_2
- removed joint joint_3
- removed joint joint_4
- removed joint joint_5
- added joint base_joint: type revolute, parent base_link, child link_1, origin xyz=0 0 0.039955 rpy=0 0 0, axis 0 0 1, limit lower=-1.5708 upper=1.5708 effort=1 velocity=1
- added joint eblow_joint: type revolute, parent link_2, child link_3, origin xyz=0 0.07545 0 rpy=0 0 0, axis 0 0 1, limit lower=-1.5708 upper=1.5708 effort=1 velocity=1
- added joint gripper_joint: type revolute, parent link_4, child link_5, origin xyz=-0.00079998 0.06655 -0.01201 rpy=0 1.5708 1.5708, axis 0 0 1, limit lower=0 upper=3.1416 effort=1 velocity=1
- added joint shoulder_joint: type revolute, parent link_1, child link_2, origin xyz=0 0 0.045445 rpy=1.5708 0 0, axis 0 0 1, limit lower=-1.5708 upper=1.5708 effort=1 velocity=1
- added joint wrist_joint: type revolute, parent link_3, child link_4, origin xyz=0 0.07545 0 rpy=0 0 0, axis 0 0 1, limit lower=-1.5708 upper=1.5708 effort=1 velocity=1
- joint joint_6: mimic joint=joint_5 multiplier=0.0062 offset=0 -> joint=gripper_joint multiplier=0.0062 offset=0
